File: Input_Power_Stage.kicad_sch (KiCad schematic)
At the start: 0 parts

Commit message: Finished 5V_Barrel over voltage red LED indicator
Parts:
- added C1: 100nF, PCM_JLCPCB:C_0603, symbol PCM_JLCPCB-Capacitors:0603,100nF
- added C2: 1uF, PCM_JLCPCB:C_0603, symbol PCM_JLCPCB-Capacitors:0603,1uF
- added C3: 1nF, PCM_JLCPCB:C_0603, symbol PCM_JLCPCB-Capacitors:0603,1nF
- added D1: 19-217/R6C-AL1M2VY/3T, LED-SMD-RED-DIFFUSED_0603_:LED-0603, symbol LED-SMD-RED-DIFFUSED_0603_:LED-SMD-RED-DIFFUSED_0603_
- added R3: 430kΩ, PCM_JLCPCB:R_0603, symbol PCM_JLCPCB-Resistors:0603,430kΩ
- added R4, R6: 100kΩ, PCM_JLCPCB:R_0603, symbol PCM_JLCPCB-Resistors:0603,100kΩ
- added R5: 82kΩ, PCM_JLCPCB:R_0603, symbol PCM_JLCPCB-Resistors:0603,82kΩ
- added R7: 360kΩ, PCM_JLCPCB:R_0603, symbol PCM_JLCPCB-Resistors:0603,360kΩ
- added R8: 3.3kΩ, PCM_JLCPCB:R_0603, symbol PCM_JLCPCB-Resistors:0603,3.3kΩ
- added U1: TPS2121RUXR, TPS2121RUXR:IC_TPS2121RUXR, symbol TPS2121RUXR:TPS2121RUXR
- added U2: AP2112K-3.3, Package_TO_SOT_SMD:SOT-23-5, symbol Regulator_Linear:AP2112K-3.3
- added U3: TLV431, symbol TLV431QFTA:TLV431QFTA
Connections:
- new net: C3.1, R6.1, R7.2, U3.1 (REF)
- new net: D1.+, R8.2, U3.3 (K)
- new net: R5.1, U1.10 (ILIM)
- new net BARREL_5V: R3.1, R7.1, R8.1, U1.2 (IN2), U1.2_1 (IN2)
- new net GND: C1.2, C2.2, C3.2, D1.-, R4.2, R5.2, R6.2, U1.12 (GND), U1.3 (CP2), U1.5 (OV1), U2.2 (GND), U3.2 (A)
- new net OV2: R3.2, R4.1, U1.4 (OV2)
- new net SS: C1.1, U1.11 (SS)
- new net ST: U1.9 (ST)
- new net SYS_3V3: U1.6 (PR1), U2.5 (VOUT)
- new net SYS_5V: C2.1, U1.1 (OUT), U1.1_1 (OUT), U1.8 (OUT), U1.8_1 (OUT), U2.1 (VIN), U2.3 (EN)
- new net VBUS_5V: U1.7 (IN1), U1.7_1 (IN1)
Other:
- company: (none) -> Yaniv Lieberman
- title: (none) -> Integrated Si5351A Module - Power Stage

Commit message: Finished Power Stage
Parts:
- added BARREL LED1: LTST-C191GKT, LTST-C191GKT:0603, symbol LTST-C191GKT:LTST-C191GKT
- added Q1, Q2, Q3: MMBT3904, Package_TO_SOT_SMD:SOT-23, symbol Transistor_BJT:MMBT3904
- added R10, R13: 100kΩ, PCM_JLCPCB:R_0603, symbol PCM_JLCPCB-Resistors:0603,100kΩ
- added R11, R12, R15: 47kΩ, PCM_JLCPCB:R_0603, symbol PCM_JLCPCB-Resistors:0603,47kΩ
- added R14, R9: 680Ω, PCM_JLCPCB:R_0603, symbol PCM_JLCPCB-Resistors:0603,680Ω
- added USB LED1: LTST-C191GKT, LTST-C191GKT:0603, symbol LTST-C191GKT:LTST-C191GKT
- OV LED1: renamed from D1
Connections:
- net GND: now also Q1.2 (E), Q2.2 (E), Q3.2 (E)
- net ST: now also R11.1, R12.1, R13.2
- net SYS_3V3: now also R10.1, R13.1, R14.1, R9.1
- new net: BARREL LED1.1, Q3.3 (C)
- new net: BARREL LED1.2, R14.2
- new net: Q2.1 (B), R12.2
- new net: Q1.3 (C), USB LED1.1
- new net: R9.2, USB LED1.2
- new net: Q3.1 (B), R15.2
- new net: Q1.1 (B), R11.2
- new net ST_INV: Q2.3 (C), R10.2, R15.1
Other:
- note added: "5V To 3.3V Voltage Regulation"
- note added: "Barrel Jack O.V LED Indicator"
- note added: "Barrel Jack O.V Threshold"
- note added: "Barrel Jack/USB LED Indicators"
- note added: "Coupling Capacitors"
- note added: "Sheet Hierarchical Pins"
- note added: "USB/Barrel Jack Power Multiplexing"
- moved on the sheet: C1, C2, C3, OV LED1, R3, R4, R5, R6, R7, R8, U1, U2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
