File: STM32 MCU Stage.kicad_sch (KiCad schematic)
At the start: 16 parts, among them J4 68000-408HLF, J5 TSM-104-01-L-SV, J6 68000-408HLF, U7 STM32G071RBT6, Y1 NX3225SA-16.000M-STD-CRS-2

Commit message: RF Module Stage Schematic Complete
Changed lines of the file:
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@@
+	(wire
+		(pts
+			(xy 22.86 57.15) (xy 26.67 57.15)
+		)
+		(stroke
+			(width 0)
+			(type default)
+		)
+	)
 	(wire
 		(pts
@@
 		)
 		(stroke
-			(width 0)
-			(type default)
-		)
-	)
-	(wire
-		(pts
-			(xy 26.67 57.15) (xy 22.86 57.15)
-		)
-		(stroke

Commit message: LCD Stage Finished
Connections:
- net SPI_MISO: no longer names the net of U7.23 (PA6)
- no-connect marks 39 -> 40

Commit message: - Added Hysteresis resistor on TLV431BSN1T1G - Lowered TLV431BSN1T1G impedance values for resistors on the voltage divider
Parts:
- J4: renamed from J5; footprint TSM-104-01-L-SV:SAMTEC_TSM-104-01-L-SV -> Samtec TSM-104-01-L-SV:SAMTEC_TSM-104-01-L-SV
- J5: renamed from J4; footprint 68000-408HLF:AMPHENOL_68000-408HLF -> 8 Pin Header - 68000-408HLF:AMPHENOL_68000-408HLF
- J6: footprint 68000-408HLF:AMPHENOL_68000-408HLF -> 8 Pin Header - 68000-408HLF:AMPHENOL_68000-408HLF
- U6: renamed from U7; footprint STM32G071RBT6:QFP50P1200X1200X160-64N -> MCU-stm32g071rbt6:QFP50P1200X1200X160-64N
- Y1: footprint NX3225SA-16.000M-STD-CRS-2:OSCCC320X250X60N -> stm32 16 mhz xtal - NX3225SA:OSCCC320X250X60N
- renumbered C17 to C19, C18 to C20, C19 to C21, C20 to C22, C21 to C23, C22 to C24, C23 to C25
Other:
- company: Yaniv Lieberman -> (none)
- title: (none) -> Integrated Si5351A Module - STM32 MCU
Changed lines of the file:
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@@
 	(paper "A4")
 	(title_block
+		(title "Integrated Si5351A Module - STM32 MCU")
 		(date "2026-02-09")
 		(rev "REV1")
-		(company "Yaniv Lieberman")
 	)
 	(rectangle
@@
 		(dnp no)
 		(fields_autoplaced yes)
-		(property "Reference" "U7"
+		(property "Reference" "U6"
 			(at 105.41 20.32 0)
 			(effects
@@
 			)
 		)
-		(property "Footprint" "STM32G071RBT6:QFP50P1200X1200X160-64N"
+		(property "Footprint" "MCU-stm32g071rbt6:QFP50P1200X1200X160-64N"
 			(at 105.41 76.2 0)
 			(effects
@@
 			(project "Integrate Si5351A Module"
 				(path "/5effc93d-4636-458a-a65b-e63d3c617be7/6855ab1b-0a54-4134-bbbf-5553693eadbf"
-					(reference "U7")
+					(reference "U6")
 					(unit 1)
 				)
@@
 		(on_board yes)
 		(dnp no)
-		(property "Reference" "C23"
+		(property "Reference" "C25"
 			(at 213.36 41.9099 0)
 			(effects
@@
 			(project "Integrate Si5351A Module"
 				(path "/5effc93d-4636-458a-a65b-e63d3c617be7/6855ab1b-0a54-4134-bbbf-5553693eadbf"
-					(reference "C23")
+					(reference "C25")
 					(unit 1)
 				)
@@
 		(on_board yes)
 		(dnp no)
-		(property "Reference" "C21"
+		(property "Reference" "C23"
 			(at 133.35 171.4499 0)
 			(effects
@@
 			(project "Integrate Si5351A Module"
 				(path "/5effc93d-4636-458a-a65b-e63d3c617be7/6855ab1b-0a54-4134-bbbf-5553693eadbf"
-					(reference "C21")
+					(reference "C23")
 					(unit 1)
 				)
@@
 		(dnp no)
 		(fields_autoplaced yes)
-		(property "Reference" "#PWR046"
+		(property "Reference" "#PWR053"
 			(at 228.6 72.39 0)
 			(effects
@@
 			(project "Integrate Si5351A Module"
 				(path "/5effc93d-4636-458a-a65b-e63d3c617be7/6855ab1b-0a54-4134-bbbf-5553693eadbf"
-					(reference "#PWR046")
+					(reference "#PWR053")
 					(unit 1)
 				)
@@
 			)
 		)
-		(property "Footprint" "NX3225SA-16.000M-STD-CRS-2:OSCCC320X250X60N"
+		(property "Footprint" "stm32 16 mhz xtal - NX3225SA:OSCCC320X250X60N"
 			(at 200.66 40.64 0)
 			(effects
@@
 		(dnp no)
 		(fields_autoplaced yes)
-		(property "Reference" "#PWR044"
+		(property "Reference" "#PWR048"
 			(at 130.81 185.42 0)
 			(effects
@@
 			(project "Integrate Si5351A Module"
 				(path "/5effc93d-4636-458a-a65b-e63d3c617be7/6855ab1b-0a54-4134-bbbf-5553693eadbf"
-					(reference "#PWR044")
+					(reference "#PWR048")
 					(unit 1)
 				)
@@
 		(dnp no)
 		(fields_autoplaced yes)
-		(property "Reference" "#PWR045"
+		(property "Reference" "#PWR049"
 			(at 158.75 80.01 0)
 			(effects
@@
 			(project "Integrate Si5351A Module"
 				(path "/5effc93d-4636-458a-a65b-e63d3c617be7/6855ab1b-0a54-4134-bbbf-5553693eadbf"
-					(reference "#PWR045")
+					(reference "#PWR049")
 					(unit 1)
 				)
@@
 		(dnp no)
 		(fields_autoplaced yes)
-		(property "Reference" "J5"
+		(property "Reference" "J4"
 			(at 187.96 81.2799 0)
 			(effects
@@
 			)
 		)
-		(property "Footprint" "TSM-104-01-L-SV:SAMTEC_TSM-104-01-L-SV"
+		(property "Footprint" "Samtec TSM-104-01-L-SV:SAMTEC_TSM-104-01-L-SV"
 			(at 181.61 81.28 0)
 			(effects
@@
 			(project "Integrate Si5351A Module"
 				(path "/5effc93d-4636-458a-a65b-e63d3c617be7/6855ab1b-0a54-4134-bbbf-5553693eadbf"
-					(reference "J5")
+					(reference "J4")
 					(unit 1)
 				)
@@
 		(dnp no)
 		(fields_autoplaced yes)
-		(property "Reference" "#PWR040"
+		(property "Reference" "#PWR044"
 			(at 66.04 87.63 0)
 			(effects
@@
 			(project "Integrate Si5351A Module"
 				(path "/5effc93d-4636-458a-a65b-e63d3c617be7/6855ab1b-0a54-4134-bbbf-5553693eadbf"
-					(reference "#PWR040")
+					(reference "#PWR044")
 					(unit 1)
 				)
@@
 		(on_board yes)
 		(dnp no)
-		(property "Reference" "C22"
+		(property "Reference" "C24"
 			(at 187.96 41.9099 0)
 			(effects
@@
 			(project "Integrate Si5351A Module"
 				(path "/5effc93d-4636-458a-a65b-e63d3c617be7/6855ab1b-0a54-4134-bbbf-5553693eadbf"
-					(reference "C22")
+					(reference "C24")
 					(unit 1)
 				)
@@
 		(on_board yes)
 		(dnp no)
-		(property "Reference" "C19"
+		(property "Reference" "C21"
 			(at 102.87 148.5899 0)
 			(effects
@@
 			(project "Integrate Si5351A Module"
 				(path "/5effc93d-4636-458a-a65b-e63d3c617be7/6855ab1b-0a54-4134-bbbf-5553693eadbf"
-					(reference "C19")
+					(reference "C21")
 					(unit 1)
 				)
@@
 		(dnp no)
 		(fields_autoplaced yes)
-		(property "Reference" "#PWR042"
+		(property "Reference" "#PWR046"
 			(at 100.33 162.56 0)
 			(effects
@@
 			(project "Integrate Si5351A Module"
 				(path "/5effc93d-4636-458a-a65b-e63d3c617be7/6855ab1b-0a54-4134-bbbf-5553693eadbf"
-					(reference "#PWR042")
+					(reference "#PWR046")
 					(unit 1)
 				)
@@
 		(dnp no)
 		(fields_autoplaced yes)
-		(property "Reference" "J4"
+		(property "Reference" "J5"
 			(at 222.25 125.7299 0)
 			(effects
@@
 			)
 		)
-		(property "Footprint" "68000-408HLF:AMPHENOL_68000-408HLF"
+		(property "Footprint" "8 Pin Header - 68000-408HLF:AMPHENOL_68000-408HLF"
 			(at 215.9 125.73 0)
 			(effects
@@
 			(project "Integrate Si5351A Module"
 				(path "/5effc93d-4636-458a-a65b-e63d3c617be7/6855ab1b-0a54-4134-bbbf-5553693eadbf"
-					(reference "J4")
+					(reference "J5")
 					(unit 1)
 				)
@@
 		(dnp no)
 		(fields_autoplaced yes)
-		(property "Reference" "#PWR041"
+		(property "Reference" "#PWR045"
 			(at 95.25 181.61 0)
 			(effects
@@
 			(project "Integrate Si5351A Module"
 				(path "/5effc93d-4636-458a-a65b-e63d3c617be7/6855ab1b-0a54-4134-bbbf-5553693eadbf"
-					(reference "#PWR041")
+					(reference "#PWR045")
 					(unit 1)
 				)
@@
 		(dnp no)
 		(fields_autoplaced yes)
-		(property "Reference" "#PWR043"
+		(property "Reference" "#PWR047"
 			(at 130.81 162.56 0)
 			(effects
@@
 			(project "Integrate Si5351A Module"
 				(path "/5effc93d-4636-458a-a65b-e63d3c617be7/6855ab1b-0a54-4134-bbbf-5553693eadbf"
-					(reference "#PWR043")
+					(reference "#PWR047")
 					(unit 1)
 				)
@@
 		(dnp no)
 		(fields_autoplaced yes)
-		(property "Reference" "#PWR048"
+		(property "Reference" "#PWR052"
 			(at 201.93 130.81 0)
 			(effects
@@
 			(project "Integrate Si5351A Module"
 				(path "/5effc93d-4636-458a-a65b-e63d3c617be7/6855ab1b-0a54-4134-bbbf-5553693eadbf"
-					(reference "#PWR048")
+					(reference "#PWR052")
 					(unit 1)
 				)
@@
 		(dnp no)
 		(fields_autoplaced yes)
-		(property "Reference" "C17"
+		(property "Reference" "C19"
 			(at 93.98 146.0499 0)
 			(effects
@@
 			(project "Integrate Si5351A Module"
 				(path "/5effc93d-4636-458a-a65b-e63d3c617be7/6855ab1b-0a54-4134-bbbf-5553693eadbf"
-					(reference "C17")
+					(reference "C19")
 					(unit 1)
 				)
@@
 		(dnp no)
 		(fields_autoplaced yes)
-		(property "Reference" "#PWR049"
+		(property "Reference" "#PWR050"
 			(at 200.66 54.61 0)
 			(effects
@@
 			(project "Integrate Si5351A Module"
 				(path "/5effc93d-4636-458a-a65b-e63d3c617be7/6855ab1b-0a54-4134-bbbf-5553693eadbf"
-					(reference "#PWR049")
+					(reference "#PWR050")
 					(unit 1)
 				)
@@
 		(on_board yes)
 		(dnp no)
-		(property "Reference" "C18"
+		(property "Reference" "C20"
 			(at 97.79 168.9099 0)
 			(effects
@@
 			(project "Integrate Si5351A Module"
 				(path "/5effc93d-4636-458a-a65b-e63d3c617be7/6855ab1b-0a54-4134-bbbf-5553693eadbf"
-					(reference "C18")
+					(reference "C20")
 					(unit 1)
 				)
@@
 		(dnp no)
 		(fields_autoplaced yes)
-		(property "Reference" "#PWR039"
+		(property "Reference" "#PWR043"
 			(at 25.4 41.91 0)
 			(effects
@@
 			(project "Integrate Si5351A Module"
 				(path "/5effc93d-4636-458a-a65b-e63d3c617be7/6855ab1b-0a54-4134-bbbf-5553693eadbf"
-					(reference "#PWR039")
+					(reference "#PWR043")
 					(unit 1)
 				)
@@
 		(dnp no)
 		(fields_autoplaced yes)
-		(property "Reference" "#PWR047"
+		(property "Reference" "#PWR051"
 			(at 201.93 119.38 0)
 			(effects
@@
 			(project "Integrate Si5351A Module"
 				(path "/5effc93d-4636-458a-a65b-e63d3c617be7/6855ab1b-0a54-4134-bbbf-5553693eadbf"
-					(reference "#PWR047")
+					(reference "#PWR051")
 					(unit 1)
 				)
@@
 		(on_board yes)
 		(dnp no)
-		(property "Reference" "C20"
+		(property "Reference" "C22"
 			(at 133.35 148.5899 0)
 			(effects
@@
 			(project "Integrate Si5351A Module"
 				(path "/5effc93d-4636-458a-a65b-e63d3c617be7/6855ab1b-0a54-4134-bbbf-5553693eadbf"
-					(reference "C20")
+					(reference "C22")
 					(unit 1)
 				)
@@
 			)
 		)
-		(property "Footprint" "68000-408HLF:AMPHENOL_68000-408HLF"
+		(property "Footprint" "8 Pin Header - 68000-408HLF:AMPHENOL_68000-408HLF"
 			(at 254 80.01 0)
 			(effects
